File: kicad/underwater.sch (KiCad schematic (older format))
At the start: 14 parts

Commit message: Add kicad net
Parts:
- removed BT?: Battery, symbol Device:Battery
- removed M? (x4): Motor_DC, symbol Motor:Motor_DC
- removed MK? (x2): IM69D130, Sensor_Audio:Infineon_PG-LLGA-5-1, symbol Sensor_Audio:IM69D130
- added BT2: Battery, Battery:BatteryHolder_Keystone_1042_1x18650, symbol Device:Battery
- added C1, C16: 3.3nF, Capacitor_SMD:C_1206_3216Metric, symbol Device:C
- added C10: 4.7μF, Capacitor_Tantalum_SMD:CP_EIA-3216-10_Kemet-I, symbol Device:CP1_Small
- added C11, C12: 0.1μF, Capacitor_Tantalum_SMD:CP_EIA-3216-10_Kemet-I, symbol Device:CP1_Small
- added C13, C14, C15, C17, C2, C20, C22: 0.1μF, Capacitor_SMD:C_1206_3216Metric, symbol Device:C
- added C18, C21, C23, C3: 10μF, Capacitor_Tantalum_SMD:CP_EIA-3216-10_Kemet-I, symbol Device:C
- added C19, C4: 22μF, Capacitor_Tantalum_SMD:CP_EIA-3216-10_Kemet-I, symbol Device:C
- added C5: 10nF, Capacitor_SMD:C_1206_3216Metric, symbol Device:C
- added C6, C7: 47pF, Capacitor_SMD:C_1206_3216Metric, symbol Device:C
- added C8, C9: 100nF, Capacitor_SMD:C_1206_3216Metric, symbol Device:C
- added D1, D2: LED_Small, LED_SMD:LED_1206_3216Metric, symbol Device:LED_Small
- added FB1: Ferrite_Bead_Small, digikey-footprints:1206, symbol Device:Ferrite_Bead_Small
- added J1, J16, J17, J18, J19, J2, J3: Screw_Terminal_01x02, TerminalBlock:TerminalBlock_bornier-2_P5.08mm, symbol Connector:Screw_Terminal_01x02
- added J10: Conn_01x05_Male, Connector_PinHeader_2.54mm:PinHeader_1x05_P2.54mm_Vertical, symbol Connector:Conn_01x05_Male
- added J11: Conn_01x06_Female, Connector_PinHeader_2.54mm:PinHeader_1x06_P2.54mm_Vertical, symbol Connector:Conn_01x06_Female
- added J12, J13, J14: Conn_01x02_Female, Connector_PinHeader_2.54mm:PinHeader_1x02_P2.54mm_Vertical, symbol Connector:Conn_01x02_Female
- added J15: Conn_01x04_Female, Connector_PinHeader_2.54mm:PinHeader_1x04_P2.54mm_Vertical, symbol Connector:Conn_01x04_Female
- added J20, J21: Conn_01x04_Female, Connector_PinHeader_2.54mm:PinHeader_1x04_P2.54mm_Horizontal, symbol Connector:Conn_01x04_Female
- added J5, J6: Conn_01x05_Female, Connector_PinHeader_2.54mm:PinHeader_1x05_P2.54mm_Vertical, symbol Connector:Conn_01x05_Female
- added J7: USB_B_Micro, digikey-footprints:USB_Micro_B_Female_10118192, symbol Connector:USB_B_Micro
- added J9: Conn_01x05_Female, Connector_PinHeader_2.54mm:PinHeader_1x05_P2.54mm_Vertical, symbol Connector:Conn_01x05_Male
- added JP1: Jumper, Jumper:SolderJumper-2_P1.3mm_Open_Pad1.0x1.5mm, symbol Device:Jumper
- added L1, L2: 2.2μH, Inductor_SMD:L_1206_3216Metric, symbol Device:L
- added MIC1, MIC2: SPH0645LM4H-B, digikey-footprints:SPH0645LM4H-B, symbol dk_Microphones:SPH0645LM4H-B
- added R1, R10: 100k, Resistor_SMD:R_1206_3216Metric, symbol Device:R
- added R11, R12: 1k, Resistor_SMD:R_1206_3216Metric, symbol Device:R
- added R2, R3: 100, Resistor_SMD:R_1206_3216Metric, symbol Device:R
- added R4, R7: 270, Resistor_SMD:R_1206_3216Metric, symbol Device:R_Small
- added R5, R6: 27, Resistor_SMD:R_1206_3216Metric, symbol Device:R
- added R8, R9: R, Resistor_SMD:R_1206_3216Metric, symbol Device:R
- added U1, U7: TPS62133, Package_DFN_QFN:VQFN-16-1EP_3x3mm_P0.5mm_EP1.68x1.68mm_ThermalVias, symbol Regulator_Switching:TPS62133
- added U2: FT230XS-U, digikey-footprints:SSOP-16_W3.90mm, symbol dk_Interface-Controllers:FT230XS-U
- added U3: LM1117-1.8, digikey-footprints:SOT-223-4, symbol Regulator_Linear:LM1117-1.8
- added U5: LM1117-3.3, digikey-footprints:SOT-223-4, symbol Regulator_Linear:LM1117-3.3
- BT1: renamed from BT?; footprint (none) -> Battery:BatteryHolder_Keystone_1042_1x18650
- J4: renamed from J?; footprint (none) -> Connector_PinHeader_2.54mm:PinHeader_1x02_P2.54mm_Vertical
- J8: renamed from J?; footprint (none) -> Connector_PinHeader_2.54mm:PinHeader_2x20_P2.54mm_Vertical
- gave numbers to parts that had none: 4
Connections:
- net at U6.10 (REGOUT): now also C15.1
- net +3V3: now reaches U6.13 (VDD)
- net +3V3: now also J8.1 (3V3), J8.2 (5V), U4.2 (VDD), UX1.13 (VM2), UX1.14 (VM3), UX1.20 (VCC), UX1.24 (VM1), UY1.13 (VM2), UY1.14 (VM3), UY1.20 (VCC), UY1.24 (VM1), C10.1, C11.1, C12.1, C14.2, C20.2, C21.2, C22.2, C23.2, C8.1, C9.1, D1.2 (A), D2.2 (A), FB1.1, J10.1 (Pin_1), J11.3 (Pin_3), J12.1 (Pin_1), J13.1 (Pin_1), J15.3 (Pin_3), J19.1 (Pin_1), J3.1 (Pin_1), J5.1 (Pin_1), J6.1 (Pin_1), J9.1 (Pin_1), JP1.1, JP1.2, MIC1.2 (SEL), MIC1.5 (VDD), MIC2.5 (VDD), R11.1, R12.1, U2.10 (3V3OUT), U2.11 (RESET), U2.12 (VCC), U2.3 (VCCIO), U3.3 (VI), U5.2 (VO), U5.3 (VI)
- net GND: now reaches U6.18 (GND), U6.20 (GND)
- net GND: now also BT1.2 (-), J8.39 (GND), J8.6 (GND), U4.1 (GND), U4.15 (GND), U4.38 (GND), UX1.10 (PGND2), UX1.18 (GND), UX1.3 (PGND1), UX1.4 (PGND1), UX1.9 (PGND2), UY1.10 (PGND2), UY1.18 (GND), UY1.3 (PGND1), UY1.4 (PGND1), UY1.9 (PGND2), BT2.2 (-), C10.2, C11.2, C12.2, C13.1, C14.1, C15.2, C17.2, C18.2, C19.2, C2.2, C20.1, C21.1, C22.1, C23.1, C3.2, C4.2, C5.2, C6.2, C7.2, C8.2, C9.2, J1.2 (Pin_2), J10.5 (Pin_5), J11.4 (Pin_4), J12.2 (Pin_2), J13.2 (Pin_2), J15.4 (Pin_4), J16.2 (Pin_2), J17.2 (Pin_2), J18.2 (Pin_2), J19.2 (Pin_2), J2.2 (Pin_2), J3.2 (Pin_2), J5.5 (Pin_5), J6.5 (Pin_5), J7.5 (GND), J7.SH (Shield), J9.5 (Pin_5), MIC1.3 (GND), MIC2.2 (SEL), MIC2.3 (GND), U1.15 (PGND), U1.16 (PGND), U1.17 (EP), U1.5 (FB), U1.6 (AGND), U1.7 (FSW), U1.8 (DEF), U2.13 (GND), U2.5 (GND), U3.1 (GND), U5.1 (GND), U7.15 (PGND), U7.16 (PGND), U7.17 (EP), U7.5 (FB), U7.6 (AGND), U7.7 (FSW), U7.8 (DEF)
- net +1V8: now reaches U6.22 (~CS)
- net +1V8: now also U6.8 (VDDIO), U6.9 (SDO/AD0), C13.2, U3.2 (VO)
- net at U6.23 (SCL/SCLK): now also U4.36 (IO22)
- net at U6.24 (SDA/SDI): now also U4.33 (IO21)
- net at UX1.1 (AO1): now also J20.1 (Pin_1)
- net at UX1.11 (BO1): now also J20.3 (Pin_3)
- net at UX1.15 (PWMB): now also U4.8 (IO32)
- net at UX1.16 (BIN2): now also U4.16 (IO13)
- net at UX1.17 (BIN1): now also U4.14 (IO12)
- net at UX1.19 (STBY): now also R11.2
- net at UX1.21 (AIN1): now also U4.12 (IO27)
- net at UX1.22 (AIN2): now also U4.37 (IO23)
- net at UX1.23 (PWMA): now also U4.10 (IO25)
- net at UX1.5 (AO2): now also J20.2 (Pin_2)
- net at UX1.7 (BO2): now also J20.4 (Pin_4)
- net at UY1.1 (AO1): now also J21.1 (Pin_1)
- net at UY1.11 (BO1): now also J21.3 (Pin_3)
- net at UY1.15 (PWMB): now also U4.9 (IO33)
- net at UY1.16 (BIN2): now also U4.26 (IO4)
- net at UY1.17 (BIN1): now also U4.27 (IO16)
- net at UY1.19 (STBY): now also R12.2
- net at UY1.21 (AIN1): now also U4.30 (IO18)
- net at UY1.22 (AIN2): now also U4.31 (IO19)
- net at UY1.23 (PWMA): now also U4.11 (IO26)
- net at UY1.5 (AO2): now also J21.2 (Pin_2)
- net at UY1.7 (BO2): now also J21.4 (Pin_4)
- net at U4.13 (IO14): now also J14.2 (Pin_2)
- net at U4.28 (IO17): now also J14.1 (Pin_1)
- net at U4.34 (RXD0/IO3): now also J15.2 (Pin_2)
- net at U4.35 (TXD0/IO1): now also J15.1 (Pin_1)
- net at J8.10 (GPIO15/RXD): now also J4.1 (Pin_1)
- net at J8.12 (GPIO18/PWM0): now also R2.2
- net at J8.35 (GPIO19/MISO1): now also R3.1
- net at J8.38 (GPIO20/MOSI1): now also J5.3 (Pin_3), J6.3 (Pin_3)
- net at J8.8 (GPIO14/TXD): now also J4.2 (Pin_2)
- net at BT1.1 (+): now also BT2.1 (+), J16.1 (Pin_1)
- new net: L1.2, U1.1 (SW), U1.2 (SW), U1.3 (SW)
- new net: C1.2, C2.1, C3.1, J2.1 (Pin_1), U1.10 (AVIN), U1.11 (PVIN), U1.12 (PVIN), U1.13 (EN)
- new net: C4.1, J1.1 (Pin_1), L1.1, R1.1, U1.14 (VOS)
- new net: R1.2, U1.4 (PG)
- new net: C1.1, U1.9 (SS/TR)
- new net: J10.2 (Pin_2), MIC1.1 (WS)
- new net: J10.4 (Pin_4), MIC1.4 (BCLK)
- new net: MIC1.6 (DATA_OUT), R8.2
- new net: J9.2 (Pin_2), MIC2.1 (WS)
- new net: J9.4 (Pin_4), MIC2.4 (BCLK)
- new net: MIC2.6 (DATA_OUT), R9.2
- new net: J10.3 (Pin_3), R8.1
- new net: J9.3 (Pin_3), R9.1
- new net: J5.2 (Pin_2), J6.2 (Pin_2), R3.2
- new net: J5.4 (Pin_4), J6.4 (Pin_4), R2.1
- new net: J11.1 (Pin_1), U2.1 (TXD)
- new net: R7.2, U2.14 (CBUS1)
- new net: J11.5 (Pin_5), U2.2 (RTS)
- new net: J11.2 (Pin_2), U2.4 (RXD)
- new net: J11.6 (Pin_6), U2.6 (CTS)
- new net: R4.2, U2.7 (CBUS2)
- new net: R5.1, U2.8 (USBDP)
- new net: R6.1, U2.9 (USBDM)
- new net: L2.2, U7.1 (SW), U7.2 (SW), U7.3 (SW)
- new net: C16.2, C17.1, C18.1, J18.1 (Pin_1), U7.10 (AVIN), U7.11 (PVIN), U7.12 (PVIN), U7.13 (EN)
- new net: C19.1, J17.1 (Pin_1), L2.1, R10.1, U7.14 (VOS)
- new net: R10.2, U7.4 (PG)
- new net: C16.1, U7.9 (SS/TR)
- new net: C5.1, FB1.2, J7.1 (VBUS)
- new net: C7.1, J7.2 (D-), R6.2
- new net: C6.1, J7.3 (D+), R5.2
- new net: D2.1 (K), R7.1
- new net: D1.1 (K), R4.1
- no-connect marks 0 -> 61
Other:
- moved on the sheet: BT1, J4, J8, U6, UX1, UY1

Commit message: Add
Parts:
- J1, J17: value Screw_Terminal_01x02 -> Batt_out
- J11: value Conn_01x06_Female -> usb_out
- J12: value Conn_01x02_Female -> esp_power5v_in
- J13: value Conn_01x02_Female -> esp_power5v_out
- J15: value Conn_01x04_Female -> usb_in
- J19: value Screw_Terminal_01x02 -> Batt_in
- J3: value Screw_Terminal_01x02 -> Power5v
- J4: value Conn_01x02_Female -> uart
Changed lines of the file:
@@
 P 750 1550
 F 0 "J4" H 778 1526 50  0000 L CNN
-F 1 "Conn_01x02_Female" H 778 1435 50  0000 L CNN
+F 1 "uart" H 778 1435 50  0000 L CNN
 F 2 "Connector_PinHeader_2.54mm:PinHeader_1x02_P2.54mm_Vertical" H 750 1550 50  0001 C CNN
 F 3 "~" H 750 1550 50  0001 C CNN
@@
 P 3650 750
 F 0 "J12" H 3678 726 50  0000 L CNN
-F 1 "Conn_01x02_Female" H 3678 635 50  0000 L CNN
+F 1 "esp_power5v_in" H 3678 635 50  0000 L CNN
 F 2 "Connector_PinHeader_2.54mm:PinHeader_1x02_P2.54mm_Vertical" H 3650 750 50  0001 C CNN
 F 3 "~" H 3650 750 50  0001 C CNN
@@
 P -500 6600
 F 0 "J1" H -420 6592 50  0000 L CNN
-F 1 "Screw_Terminal_01x02" H -420 6501 50  0000 L CNN
+F 1 "Batt_out" H -420 6501 50  0000 L CNN
 F 2 "TerminalBlock:TerminalBlock_bornier-2_P5.08mm" H -500 6600 50  0001 C CNN
 F 3 "~" H -500 6600 50  0001 C CNN
@@
 P 8650 9750
 F 0 "J17" H 8730 9742 50  0000 L CNN
-F 1 "Screw_Terminal_01x02" H 8730 9651 50  0000 L CNN
+F 1 "Batt_out" H 8730 9651 50  0000 L CNN
 F 2 "TerminalBlock:TerminalBlock_bornier-2_P5.08mm" H 8650 9750 50  0001 C CNN
 F 3 "~" H 8650 9750 50  0001 C CNN
@@
 P 8950 6200
 F 0 "J19" V 8822 6280 50  0000 L CNN
-F 1 "Screw_Terminal_01x02" V 8913 6280 50  0000 L CNN
+F 1 "Batt_in" V 8913 6280 50  0000 L CNN
 F 2 "TerminalBlock:TerminalBlock_bornier-2_P5.08mm" H 8950 6200 50  0001 C CNN
 F 3 "~" H 8950 6200 50  0001 C CNN
@@
 P 7450 100
 F 0 "J15" V 7388 -188 50  0000 R CNN
-F 1 "Conn_01x04_Female" V 7297 -188 50  0000 R CNN
+F 1 "usb_in" V 7297 -188 50  0000 R CNN
 F 2 "Connector_PinHeader_2.54mm:PinHeader_1x04_P2.54mm_Vertical" H 7450 100 50  0001 C CNN
 F 3 "~" H 7450 100 50  0001 C CNN
@@
 P 4350 -200
 F 0 "J13" H 4242 -525 50  0000 C CNN
-F 1 "Conn_01x02_Female" H 4242 -434 50  0000 C CNN
+F 1 "esp_power5v_out" H 4242 -434 50  0000 C CNN
 F 2 "Connector_PinHeader_2.54mm:PinHeader_1x02_P2.54mm_Vertical" H 4350 -200 50  0001 C CNN
 F 3 "~" H 4350 -200 50  0001 C CNN
@@
 P 2950 5250
 F 0 "J11" V 2888 4862 50  0000 R CNN
-F 1 "Conn_01x06_Female" V 2797 4862 50  0000 R CNN
+F 1 "usb_out" V 2797 4862 50  0000 R CNN
 F 2 "Connector_PinHeader_2.54mm:PinHeader_1x06_P2.54mm_Vertical" H 2950 5250 50  0001 C CNN
 F 3 "~" H 2950 5250 50  0001 C CNN
@@
 P 750 950
 F 0 "J3" H 668 625 50  0000 C CNN
-F 1 "Screw_Terminal_01x02" H 668 716 50  0000 C CNN
+F 1 "Power5v" H 668 716 50  0000 C CNN
 F 2 "TerminalBlock:TerminalBlock_bornier-2_P5.08mm" H 750 950 50  0001 C CNN
 F 3 "~" H 750 950 50  0001 C CNN
