File: kicad/underwater.kicad_pcb (KiCad board)
At the start: 2 copper layers, 75 parts, among them J1 Screw_Terminal_01x02, J10 Conn_01x05_Male, J11 Conn_01x06_Female, J12 Conn_01x02_Female, J13 Conn_01x02_Female, J14 Conn_01x02_Female, J15 Conn_01x04_Female, J16 Screw_Terminal_01x02, J17 Screw_Terminal_01x02, J18 Screw_Terminal_01x02, J19 Screw_Terminal_01x02, J2 Screw_Terminal_01x02, J20 Conn_01x04_Female, J21 Conn_01x04_Female, J3 Screw_Terminal_01x02, J4 Conn_01x02_Female, J5 Conn_01x05_Female, J6 Conn_01x05_Female, J7 USB_B_Micro, J8 Raspberry_Pi_2_3, J9 Conn_01x05_Female, U1 TPS62133, U2 FT230XS-U, U3 LM1117-1.8, U4 ESP32-WROOM-32, U5 LM1117-3.3, U6 ICM-20948, U7 TPS62133

Commit message: Add
Parts:
- J1, J17: value Screw_Terminal_01x02 -> Batt_out
- J11: value Conn_01x06_Female -> usb_out
- J12: value Conn_01x02_Female -> esp_power5v_in
- J13: value Conn_01x02_Female -> esp_power5v_out
- J15: value Conn_01x04_Female -> usb_in
- J19: value Screw_Terminal_01x02 -> Batt_in
- J3: value Screw_Terminal_01x02 -> Power5v
- J4: value Conn_01x02_Female -> uart
- moved J3 4.02 mm to (130.8, 34.3)
- moved J4 4.02 mm to (134.6, 52.1)
- moved J8 4.02 mm to (127.0, 41.9)
- moved R2 4.02 mm to (133.3, 57.1)
- moved J12 4.02 mm to (134.6, 40.6)
- moved J5 4.02 mm to (123.2, 100.3)
- moved J6 4.02 mm to (123.2, 96.4)
- moved R3 4.02 mm to (123.2, 86.4)
- moved C12 3.59 mm to (106.6, 49.5)
- moved MIC1 3.59 mm to (106.0, 54.6)
- moved MIC2 3.59 mm to (106.0, 36.8)
- moved C11 3.59 mm to (106.8, 31.8)
- moved J10 3.59 mm to (116.8, 49.5)
- moved J9 3.59 mm to (116.8, 31.8)
- moved R8 3.59 mm to (113.0, 54.6)
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Routing:
- net +3V3: track 183.4 -> 256.7 mm, vias 6 -> 10
- net GND: track 512.0 -> 537.1 mm, vias 14 -> 16
- net Net-(J5-Pad3): track 3.94 -> 16.1 mm
Other:
- board outline added: 179.1 x 124.5 mm

Commit message: fix
Parts:
- moved J16 114.0 mm to (230.5, 88.9)
- moved BT1 114.0 mm to (216.5, 45.7)
- moved BT2 114.0 mm to (239.4, 45.7)
- moved C20 94.0 mm to (173.4, 70.5)
- moved R12 94.0 mm to (184.8, 70.5)
- moved C13 94.0 mm to (153.0, 65.4)
- moved C14 94.0 mm to (158.1, 65.5)
- moved C15 94.0 mm to (163.2, 65.4)
- moved C21 94.0 mm to (178.4, 70.6)
- moved C22 94.0 mm to (194.9, 70.6)
- moved C23 94.0 mm to (189.9, 70.5)
- moved J13 94.0 mm to (149.2, 45.1)
- moved J14 94.0 mm to (187.3, 60.3)
- moved J15 94.0 mm to (187.3, 43.8)
- moved J20 94.0 mm to (164.5, 94.6)
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Routing:
- net GND: track 537.1 -> 667.7 mm, vias 16 -> 21
- net Net-(U4-Pad36): track 0.00 -> 73.3 mm, vias 0 -> 6
- net Net-(U4-Pad33): track 0.00 -> 67.7 mm, vias 0 -> 4
- net Net-(U4-Pad37): track 0.00 -> 57.3 mm, vias 0 -> 4
- net Net-(J14-Pad2): track 0.00 -> 45.9 mm, vias 0 -> 4
- net Net-(U4-Pad9): track 8.10 -> 48.4 mm, vias 1 -> 2
- net Net-(U4-Pad11): track 0.00 -> 37.3 mm, vias 0 -> 2
- net Net-(U4-Pad10): track 1.25 -> 30.5 mm, vias 0 -> 2
- net Net-(U4-Pad12): track 0.00 -> 27.8 mm, vias 0 -> 2
- net Net-(U4-Pad8): track 9.46 -> 32.2 mm, vias 1 -> 2
- net Net-(U4-Pad14): track 0.00 -> 21.5 mm, vias 0 -> 2
- net Net-(J21-Pad1): track 0.00 -> 13.1 mm, vias 0 -> 2
- net Net-(J21-Pad2): track 0.00 -> 11.7 mm, vias 0 -> 2
- net Net-(J14-Pad1): track 0.00 -> 11.0 mm
- net Net-(J15-Pad1): track 0.00 -> 10.2 mm, vias 0 -> 1
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Other:
- board size 179.1 x 124.5 mm -> 135.3 x 141.6 mm

Commit message: Fix
Parts:
- moved J17 79.5 mm to (151.1, 104.8), turned to 0 degrees
- moved C19 68.6 mm to (153.7, 113.7), turned to 90 degrees
- moved J18 68.4 mm to (162.6, 104.8), turned to 0 degrees
- moved L2 66.8 mm to (151.1, 120.1), turned to 270 degrees
- moved C18 63.1 mm to (158.8, 113.7), turned to 90 degrees
- moved J1 59.6 mm to (175.4, 104.9), turned to 0 degrees
- moved R10 58.0 mm to (155.1, 126.4), turned to 0 degrees
- moved U7 56.7 mm to (158.8, 121.3), turned to 90 degrees
- moved C17 56.4 mm to (165.1, 113.8), turned to 90 degrees
- moved J2 55.1 mm to (186.4, 104.8), turned to 0 degrees
- moved C16 50.4 mm to (165.1, 120.0), turned to 90 degrees
- moved C4 46.2 mm to (178.4, 113.7), turned to 90 degrees
- moved C3 43.8 mm to (183.5, 113.7), turned to 90 degrees
- moved C2 42.4 mm to (188.6, 113.7), turned to 90 degrees
- moved L1 39.9 mm to (175.9, 120.1), turned to 270 degrees
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Routing:
- net +3V3: track 256.7 -> 432.8 mm, vias 10 -> 22
- net Net-(U4-Pad31): track 0.00 -> 36.8 mm, vias 0 -> 2
- net Net-(U4-Pad30): track 0.00 -> 35.7 mm, vias 0 -> 2
- net Net-(U4-Pad27): track 0.00 -> 30.3 mm, vias 0 -> 2
- net Net-(U4-Pad26): track 0.00 -> 28.1 mm, vias 0 -> 2
- net Net-(R12-Pad2): track 0.00 -> 12.9 mm
- net Net-(C5-Pad1): track 4.33 -> 17.1 mm, vias 0 -> 2
- net Net-(U4-Pad36): track 73.3 -> 78.3 mm
- net Net-(R11-Pad2): track 14.6 -> 17.8 mm
- net Net-(U4-Pad37): track 57.3 -> 59.6 mm
- net Net-(U4-Pad33): track 67.7 -> 65.6 mm
- net GND: track 667.7 -> 669.4 mm
- net Net-(J14-Pad2): track 45.9 -> 44.4 mm
- net +1V8: track 16.0 -> 17.3 mm
- net Net-(U4-Pad12): track 27.8 -> 26.5 mm
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- added copper zone on F.Cu, net GND
Other:
- board size 135.3 x 141.6 mm -> 93.3 x 102.2 mm

Commit message: format
Parts:
- removed BT1, BT2: Battery, Battery:BatteryHolder_Keystone_1042_1x18650
- removed J16: Screw_Terminal_01x02, TerminalBlock:TerminalBlock_bornier-2_P5.08mm
- added REF**: OSHW-Logo_11.4x12mm_SilkScreen, Symbol:OSHW-Logo_11.4x12mm_SilkScreen, F.Cu at (148.6, 87.1)
- moved C10 3.81 mm to (136.5, 126.4)
- moved C5 3.81 mm to (111.1, 126.4)
- moved C6 3.81 mm to (116.2, 126.4)
- moved C7 3.81 mm to (121.3, 126.4)
- moved D1 3.81 mm to (146.7, 114.9)
- moved D2 3.81 mm to (146.8, 120.0)
- moved FB1 3.81 mm to (115.7, 111.1)
- moved J11 3.81 mm to (146.7, 108.6)
- moved R4 3.81 mm to (141.6, 114.9)
- moved R5 3.81 mm to (117.6, 117.5)
- moved R6 3.81 mm to (122.7, 114.9)
- moved R7 3.81 mm to (141.7, 120.0)
- moved C8 3.81 mm to (126.4, 126.4)
- moved C9 3.81 mm to (131.4, 126.4)
- moved J7 3.81 mm to (108.6, 114.9)
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Routing:
- net GND: track 669.4 -> 563.3 mm, vias 21 -> 20
- net Net-(BT1-Pad1): track 26.3 -> 0.00 mm
Other:
- board size 93.3 x 102.2 mm -> 94.6 x 99.8 mm

Commit message: Fix
Parts:
- moved MIC2 1.42 mm to (108.6, 40.0)
- moved R9 1.42 mm to (115.6, 39.9)
- moved C12 1.42 mm to (109.1, 52.7)
- moved MIC1 1.42 mm to (108.6, 57.8)
- moved C11 1.42 mm to (109.3, 34.9)
- moved J10 1.42 mm to (119.4, 52.7)
- moved J9 1.42 mm to (119.4, 34.9)
- moved R8 1.42 mm to (115.6, 57.8)
Routing:
- net GND: track 563.3 -> 602.0 mm
- net +3V3: track 432.8 -> 468.9 mm, vias 22 -> 25
- net +1V8: track 17.3 -> 29.9 mm, vias 0 -> 2
- net Net-(C1-Pad2): track 35.0 -> 42.6 mm
- net Net-(R5-Pad1): track 25.2 -> 22.2 mm
- net Net-(R7-Pad2): track 20.5 -> 23.1 mm
- net Net-(L1-Pad2): track 8.29 -> 10.8 mm
- net Net-(C7-Pad1): track 20.3 -> 20.9 mm
Other:
- board size 94.6 x 99.8 mm -> 93.3 x 97.2 mm
